File: board/servo_board/servo_board.kicad_pcb (KiCad board)
At the start: 2 copper layers, 72.4 x 60.3 mm, 52 parts, among them J1 knee_right, J10 box1_up, J11 box2_up, J12 Power_input, J13 body_right_up, J14 Left_ESP32, J15 Right_ESP32, J16 Conn_01x11_Male, J17 Conn_01x11_Male, J18 Conn_01x02_Female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

Commit message: UpdatePCB gerber
Parts:
- added C4: 470uF, Capacitor_SMD:CP_Elec_6.3x7.7, F.Cu at (137.5, 157.1)
- added R22: 220, Resistor_SMD:R_1206_3216Metric_Pad1.30x1.75mm_HandSolder, F.Cu at (137.3, 167.0)
- added R23: 220, Resistor_SMD:R_1206_3216Metric_Pad1.30x1.75mm_HandSolder, F.Cu at (141.0, 167.0)
- C1: value 1000uF -> 470uF; footprint Capacitor_SMD:CP_Elec_10x10.5 -> Capacitor_SMD:CP_Elec_6.3x7.7
- R17, R18: value 10k -> 2.2k
- moved J22 166.4 mm to (105.0, 173.7), turned to 0 degrees
- moved J9 164.8 mm to (101.4, 173.7), turned to 0 degrees
- moved J1 163.3 mm to (97.8, 173.7), turned to 0 degrees
- moved J21 161.9 mm to (94.2, 173.7), turned to 0 degrees
- moved J8 160.7 mm to (90.6, 173.7), turned to 0 degrees
- moved J2 159.6 mm to (87.0, 173.7), turned to 0 degrees
- moved R1 151.1 mm to (87.0, 167.4), turned to 270 degrees
- moved J13 149.5 mm to (83.5, 173.7), turned to 0 degrees
- moved R2 147.6 mm to (90.7, 167.4), turned to 270 degrees
- moved J24 145.6 mm to (108.6, 173.7), turned to 0 degrees
- moved R6 144.2 mm to (94.3, 167.5), turned to 270 degrees
- moved J11 142.0 mm to (112.2, 173.7), turned to 0 degrees
- moved R5 140.9 mm to (98.0, 167.3), turned to 270 degrees
- moved D1 139.8 mm to (93.0, 153.8)
- moved J6 138.3 mm to (115.8, 173.7), turned to 0 degrees
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Connections:
- J14 pad 3: right_wrist -> Net-(J14-Pad3)
- J15 pad 11: right_shoulder -> Net-(J15-Pad11)
- J15 pad 15: VIN -> +5V
- J17 pad 11: VIN -> +5V
Routing:
- net GND: track 403.8 -> 202.8 mm
- net +5V: track 181.3 -> 278.3 mm
- net D13: track 4.67 -> 98.0 mm
- net D12: track 4.67 -> 91.5 mm
- net D27: track 4.26 -> 82.7 mm
- net Net-(J14-Pad3): track 0.00 -> 72.5 mm
- net right_wrist: track 77.5 -> 5.18 mm
- net D26: track 4.26 -> 76.5 mm
- net D25: track 4.26 -> 70.3 mm
- net D33: track 4.26 -> 64.1 mm
- net D32: track 4.26 -> 57.9 mm
- net D35: track 4.26 -> 51.7 mm
- net D34: track 4.26 -> 45.5 mm
- net TX0: track 4.82 -> 45.8 mm
- net Net-(J15-Pad11): track 0.00 -> 40.2 mm
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- added copper zone on B.Cu, net GND
Other:
- board size 72.4 x 60.3 mm -> 81.5 x 96.5 mm
- board text added: "+5V"
- board text added: "0"
- board text added: "1"
- board text added: "10"
- board text added: "11"
- board text added: "12"
- board text added: "13"
- board text added: "14"
- board text added: "15"
- board text added: "16"
- board text added: "17"
- board text added: "2"
- board text added: "3"
- board text added: "4"
- board text added: "5"
- board text added: "6"
- board text added: "7"
- board text added: "8"
- board text added: "9"
- board text added: "ESP32-PCA Robot Board V0.1"
- board text added: "by Jip"
- board text removed: "3.3V"
- board text removed: "BRU"
- board text removed: "RS"
- board text removed: "RW"
- board text removed: "SCL"
- board text removed: "SDA"
- board text removed: "VIN"
